File: Hardware/PrototypeBoard/MainConnector.sch (KiCad schematic (older format))
At the start: 13 parts, among them J3 ControlSupplyConnector

Commit message: Migrated to kicad 5
Parts:
- C34, C35, C36, C37, C38, C39, C40: symbol C -> Device:C
- D7, D8, D9: symbol D_TVS -> Device:D_TVS
- F1, F2: symbol Fuse -> Device:Fuse
- J3: symbol Conn_02x24_Odd_Even -> conn:Conn_02x24_Odd_Even
Changed lines of the file:
@@
-EESchema Schematic File Version 2
-LIBS:power
-LIBS:device
-LIBS:switches
-LIBS:relays
-LIBS:motors
-LIBS:transistors
-LIBS:conn
-LIBS:linear
-LIBS:regul
-LIBS:74xx
-LIBS:cmos4000
-LIBS:adc-dac
-LIBS:memory
-LIBS:xilinx
-LIBS:microcontrollers
-LIBS:dsp
-LIBS:microchip
-LIBS:analog_switches
-LIBS:motorola
-LIBS:texas
-LIBS:intel
-LIBS:audio
-LIBS:interface
-LIBS:digital-audio
-LIBS:philips
-LIBS:display
-LIBS:cypress
-LIBS:siliconi
-LIBS:opto
-LIBS:atmel
-LIBS:contrib
-LIBS:valves
+EESchema Schematic File Version 4
 LIBS:PrototypeBoard-cache
-EELAYER 25 0
+EELAYER 26 0
 EELAYER END
 $Descr A4 11693 8268
@@
 CurrentSensSpiDoutW
 $Comp
-L Conn_02x24_Odd_Even J3
+L conn:Conn_02x24_Odd_Even J3
 U 1 1 5AFFC4D2
 P 4000 3400
@@
 $EndComp
 $Comp
-L GNDPWR #PWR069
+L PrototypeBoard-rescue:GNDPWR #PWR069
 U 1 1 5AFFC52B
 P 3600 4600
@@
 $EndComp
 $Comp
-L GNDPWR #PWR070
+L PrototypeBoard-rescue:GNDPWR #PWR070
 U 1 1 5AFFC541
 P 3600 2300
@@
 $EndComp
 $Comp
-L +BATT #PWR071
+L power:+BATT #PWR071
 U 1 1 5AFFC5BD
 P 8200 2300
@@
 $EndComp
 $Comp
-L GND #PWR072
+L power:GND #PWR072
 U 1 1 5AFFC6F4
 P 3600 2600
@@
 $EndComp
 $Comp
-L GND #PWR073
+L power:GND #PWR073
 U 1 1 5AFFC70F
 P 3600 4300
@@
 $EndComp
 $Comp
-L +3.3V #PWR074
+L power:+3.3V #PWR074
 U 1 1 5AFFC799
 P 6700 2600
@@
 $EndComp
 $Comp
-L GND #PWR075
+L power:GND #PWR075
 U 1 1 5AFFCA44
 P 3600 4100
@@
 $EndComp
 $Comp
-L GND #PWR076
+L power:GND #PWR076
 U 1 1 5AFFCA52
 P 3600 4000
@@
 $EndComp
 $Comp
-L GND #PWR077
+L power:GND #PWR077
 U 1 1 5AFFCA60
 P 3600 3900
@@
 $EndComp
 $Comp
-L GND #PWR078
+L power:GND #PWR078
 U 1 1 5AFFCA6E
 P 3600 3700
@@
 $EndComp
 $Comp
-L GND #PWR079
+L power:GND #PWR079
 U 1 1 5AFFCA7C
 P 3600 3600
@@
 $EndComp
 $Comp
-L GND #PWR080
+L power:GND #PWR080
 U 1 1 5AFFCA98
 P 3600 3500
@@
 $EndComp
 $Comp
-L GND #PWR081
+L power:GND #PWR081
 U 1 1 5AFFCAA6
 P 3600 3400
@@
 $EndComp
 $Comp
-L GND #PWR082
+L power:GND #PWR082
 U 1 1 5AFFCAB4
 P 3600 3200
@@
 $EndComp
 $Comp
-L Fuse F2
+L Device:Fuse F2
 U 1 1 5B0008BD
 P 7450 2300
@@
 $EndComp
 $Comp
-L +3.3V #PWR083
+L power:+3.3V #PWR083
 U 1 1 5AFF6F2E
 P 3600 5900
@@
 $EndComp
 $Comp
-L PWR_FLAG #FLG084
+L power:PWR_FLAG #FLG084
 U 1 1 5AFF6F6D
 P 3600 6100
@@
 $EndComp
 $Comp
-L PWR_FLAG #FLG085
+L power:PWR_FLAG #FLG085
 U 1 1 5AFF70D3
 P 4600 5900
@@
 Connection ~ 4400 2400
 $Comp
-L PWR_FLAG #FLG086
+L power:PWR_FLAG #FLG086
 U 1 1 5AFF727E
 P 4100 6100
@@
 $EndComp
 $Comp
-L +BATT #PWR087
+L power:+BATT #PWR087
 U 1 1 5AFF72BB
 P 4100 5900
@@
 	4100 5900 4100 6100
 $Comp
-L GND #PWR088
+L power:GND #PWR088
 U 1 1 5AFF731E
 P 4600 6100
@@
 	4600 5900 4600 6100
 $Comp
-L PWR_FLAG #FLG089
+L power:PWR_FLAG #FLG089
 U 1 1 5AFF7374
 P 5100 5900
@@
 $EndComp
 $Comp
-L GNDPWR #PWR090
+L PrototypeBoard-rescue:GNDPWR #PWR090
 U 1 1 5AFF7385
 P 5100 6100
@@
 	4300 2800 4500 2800
 $Comp
-L GND #PWR091
+L power:GND #PWR091
 U 1 1 5AFF86D9
 P 3600 2800
@@
 	3600 2800 3800 2800
 $Comp
-L C C34
+L Device:C C34
 U 1 1 5AFF8734
 P 4050 1700
@@
 $EndComp
 $Comp
-L C C37
+L Device:C C37
 U 1 1 5AFF8906
 P 4050 5200
@@
 Since ERC complains about no drivers in power net \n(connector pins don't have the type "Power Output"), \nthis workaround has to be used
 $Comp
-L GNDPWR #PWR092
+L PrototypeBoard-rescue:GNDPWR #PWR092
 U 1 1 5B0080B7
 P 7900 2800
@@
 Connection ~ 7200 2300
 $Comp
-L Fuse F1
+L Device:Fuse F1
 U 1 1 5B00839B
 P 6150 2600
@@
 Connection ~ 5900 3900
 $Comp
-L GND #PWR093
+L power:GND #PWR093
 U 1 1 5B008FFB
 P 6500 3100
@@
 $EndComp
 $Comp
-L D_TVS D9
+L Device:D_TVS D9
 U 1 1 5B00D2A4
 P 7900 2550
@@
 	7900 2700 7900 2800
 $Comp
-L D_TVS D7
+L Device:D_TVS D7
 U 1 1 5B00D572
 P 6500 2850
@@
 Connection ~ 6500 2600
 $Comp
-L C C36
+L Device:C C36
 U 1 1 5B00D7DF
 P 4050 4900
@@
 Connection ~ 3700 4900
 $Comp
-L C C35
+L Device:C C35
 U 1 1 5B00D9FF
 P 4050 2000
@@
 Connection ~ 4400 2000
 $Comp
-L C C38
+L Device:C C38
 U 1 1 5B00DC69
 P 5800 2850
@@
 $EndComp
 $Comp
-L C C39
+L Device:C C39
 U 1 1 5B00DD38
 P 6150 3900
@@
 $EndComp
 $Comp
-L C C40
+L Device:C C40
 U 1 1 5B00DD8B
 P 6150 4300
@@
 Connection ~ 5900 4300
 $Comp
-L GND #PWR094
+L power:GND #PWR094
 U 1 1 5B00DFF3
 P 6400 3900
@@
 $EndComp
 $Comp
-L GND #PWR095
+L power:GND #PWR095
 U 1 1 5B00E052
 P 6400 4300
@@
 Connection ~ 5800 2600
 $Comp
-L GND #PWR096
+L power:GND #PWR096
 U 1 1 5B00E24D
 P 5800 3100
@@
 3V3in
 $Comp
-L D_TVS D8
+L Device:D_TVS D8
 U 1 1 5B27A7EB
 P 7000 2450
@@
 Connection ~ 7000 2300
 $Comp
-L GNDPWR #PWR097
+L PrototypeBoard-rescue:GNDPWR #PWR097
 U 1 1 5B27AA44
 P 7000 2650
