File: Hardware/PrototypeBoard/Adc.sch (KiCad schematic (older format))
At the start: 29 parts, among them U5 ADC124S021

Commit message: some more layout...
Parts:
- added R26: 0, Resistors_SMD:R_0805_HandSoldering, symbol R
- renumbered C24 to C27, C25 to C28, C26 to C29, C27 to C30, C28 to C31, C29 to C32, R26 to R27, R27 to R28, R28 to R29, R29 to R30, R30 to R31, R31 to R32, R32 to R33, R33 to R34
Connections:
- net +3V3: now also R26.2; no longer L1.1
- new net: L1.1, R26.1
Changed lines of the file:
@@
 $EndComp
 $Comp
-L C C25
+L C C28
 U 1 1 5AFC7ED4
 P 2400 3100
-F 0 "C25" H 2425 3200 50  0000 L CNN
+F 0 "C28" H 2425 3200 50  0000 L CNN
 F 1 "100n" H 2425 3000 50  0000 L CNN
 F 2 "Capacitors_SMD:C_0805_HandSoldering" H 2438 2950 50  0001 C CNN
@@
 $EndComp
 $Comp
-L C C24
+L C C27
 U 1 1 5AFC7FC0
 P 2150 3100
-F 0 "C24" H 2175 3200 50  0000 L CNN
+F 0 "C27" H 2175 3200 50  0000 L CNN
 F 1 "1μ" H 2175 3000 50  0000 L CNN
 F 2 "Capacitors_SMD:C_0805_HandSoldering" H 2188 2950 50  0001 C CNN
@@
 L +3.3V #PWR049
 U 1 1 5AFC801E
-P 1700 3250
-F 0 "#PWR049" H 1700 3100 50  0001 C CNN
-F 1 "+3.3V" H 1700 3390 50  0000 C CNN
-F 2 "" H 1700 3250 50  0001 C CNN
-F 3 "" H 1700 3250 50  0001 C CNN
-	1    1700 3250
-	1    0    0    -1
-$EndComp
-Wire Wire Line
-	1700 3250 1750 3250
+P 1350 3250
+F 0 "#PWR049" H 1350 3100 50  0001 C CNN
+F 1 "+3.3V" H 1350 3390 50  0000 C CNN
+F 2 "" H 1350 3250 50  0001 C CNN
+F 3 "" H 1350 3250 50  0001 C CNN
+	1    1350 3250
+	1    0    0    -1
+$EndComp
 Text HLabel 1900 3400 0    60   Input ~ 0
 ~CS
@@
 	1900 3700 3200 3700
 $Comp
-L C C29
+L C C32
 U 1 1 5AFD651F
 P 9900 4050
-F 0 "C29" H 9925 4150 50  0000 L CNN
+F 0 "C32" H 9925 4150 50  0000 L CNN
 F 1 "DNP" H 9925 3950 50  0000 L CNN
 F 2 "Capacitors_SMD:C_0805_HandSoldering" H 9938 3900 50  0001 C CNN
@@
 $EndComp
 $Comp
-L C C28
+L C C31
 U 1 1 5AFD65A4
 P 8500 4050
-F 0 "C28" H 8525 4150 50  0000 L CNN
+F 0 "C31" H 8525 4150 50  0000 L CNN
 F 1 "DNP" H 8525 3950 50  0000 L CNN
 F 2 "Capacitors_SMD:C_0805_HandSoldering" H 8538 3900 50  0001 C CNN
@@
 $EndComp
 $Comp
-L C C27
+L C C30
 U 1 1 5AFD65D2
 P 7100 4050
-F 0 "C27" H 7125 4150 50  0000 L CNN
+F 0 "C30" H 7125 4150 50  0000 L CNN
 F 1 "DNP" H 7125 3950 50  0000 L CNN
 F 2 "Capacitors_SMD:C_0805_HandSoldering" H 7138 3900 50  0001 C CNN
@@
 $EndComp
 $Comp
-L C C26
+L C C29
 U 1 1 5AFD660C
 P 5700 4050
-F 0 "C26" H 5725 4150 50  0000 L CNN
+F 0 "C29" H 5725 4150 50  0000 L CNN
 F 1 "100n" H 5725 3950 50  0000 L CNN
 F 2 "Capacitors_SMD:C_0805_HandSoldering" H 5738 3900 50  0001 C CNN
@@
 $EndComp
 $Comp
-L R R26
+L R R27
 U 1 1 5AFD665A
 P 6000 3050
-F 0 "R26" V 6080 3050 50  0000 C CNN
+F 0 "R27" V 6080 3050 50  0000 C CNN
 F 1 "8.2k" V 6000 3050 50  0000 C CNN
 F 2 "Resistors_SMD:R_0805_HandSoldering" V 5930 3050 50  0001 C CNN
@@
 $EndComp
 $Comp
-L R R28
+L R R29
 U 1 1 5AFD6721
 P 7400 3050
-F 0 "R28" V 7480 3050 50  0000 C CNN
+F 0 "R29" V 7480 3050 50  0000 C CNN
 F 1 "6.8k" V 7400 3050 50  0000 C CNN
 F 2 "Resistors_SMD:R_0805_HandSoldering" V 7330 3050 50  0001 C CNN
@@
 $EndComp
 $Comp
-L R R30
+L R R31
 U 1 1 5AFD6757
 P 8800 3050
-F 0 "R30" V 8880 3050 50  0000 C CNN
+F 0 "R31" V 8880 3050 50  0000 C CNN
 F 1 "6.8k" V 8800 3050 50  0000 C CNN
 F 2 "Resistors_SMD:R_0805_HandSoldering" V 8730 3050 50  0001 C CNN
@@
 $EndComp
 $Comp
-L R R32
+L R R33
 U 1 1 5AFD6790
 P 10200 3050
-F 0 "R32" V 10280 3050 50  0000 C CNN
+F 0 "R33" V 10280 3050 50  0000 C CNN
 F 1 "6.8k" V 10200 3050 50  0000 C CNN
 F 2 "Resistors_SMD:R_0805_HandSoldering" V 10130 3050 50  0001 C CNN
@@
 	10200 2800 10200 2900
 $Comp
-L R R33
+L R R34
 U 1 1 5AFD684A
 P 10200 4050
-F 0 "R33" V 10280 4050 50  0000 C CNN
+F 0 "R34" V 10280 4050 50  0000 C CNN
 F 1 "DNP" V 10200 4050 50  0000 C CNN
 F 2 "Resistors_SMD:R_0805_HandSoldering" V 10130 4050 50  0001 C CNN
@@
 $EndComp
 $Comp
-L R R31
+L R R32
 U 1 1 5AFD68B5
 P 8800 4050
-F 0 "R31" V 8880 4050 50  0000 C CNN
+F 0 "R32" V 8880 4050 50  0000 C CNN
 F 1 "1k" V 8800 4050 50  0000 C CNN
 F 2 "Resistors_SMD:R_0805_HandSoldering" V 8730 4050 50  0001 C CNN
@@
 $EndComp
 $Comp
-L R R29
+L R R30
 U 1 1 5AFD6903
 P 7400 4050
-F 0 "R29" V 7480 4050 50  0000 C CNN
+F 0 "R30" V 7480 4050 50  0000 C CNN
 F 1 "1k" V 7400 4050 50  0000 C CNN
 F 2 "Resistors_SMD:R_0805_HandSoldering" V 7330 4050 50  0001 C CNN
@@
 $EndComp
 $Comp
-L R R27
+L R R28
 U 1 1 5AFD695A
 P 6000 4050
-F 0 "R27" V 6080 4050 50  0000 C CNN
+F 0 "R28" V 6080 4050 50  0000 C CNN
 F 1 "1k" V 6000 4050 50  0000 C CNN
 F 2 "Resistors_SMD:R_0805_HandSoldering" V 5930 4050 50  0001 C CNN
@@
 	0    1    1    0
 $EndComp
+$Comp
+L R R26
+U 1 1 5B210B75
+P 1550 3250
+F 0 "R26" V 1630 3250 50  0000 C CNN
+F 1 "0" V 1550 3250 50  0000 C CNN
+F 2 "Resistors_SMD:R_0805_HandSoldering" V 1480 3250 50  0001 C CNN
+F 3 "" H 1550 3250 50  0001 C CNN
+	1    1550 3250
+	0    1    1    0
+$EndComp
+Wire Wire Line
+	1350 3250 1400 3250
+Wire Wire Line
+	1700 3250 1750 3250
 $EndSCHEMATC

Commit message: more layout and some changes to schematic
Parts:
- TP22, TP23, TP24, TP25, TP26, TP27, TP28, TP29, TP30: footprint Measurement_Points:Measurement_Point_Round-SMD-Pad_Small -> Pin_Headers:Pin_Header_Straight_1x01_Pitch2.00mm
Changed lines of the file:
@@
 F 0 "TP27" H 5100 4200 50  0000 C BNN
 F 1 "Adc4" H 5100 4150 50  0000 C CNN
-F 2 "Measurement_Points:Measurement_Point_Round-SMD-Pad_Small" H 5100 3900 50  0001 C CNN
+F 2 "Pin_Headers:Pin_Header_Straight_1x01_Pitch2.00mm" H 5100 3900 50  0001 C CNN
 F 3 "" H 5100 3900 50  0001 C CNN
 	1    5100 3900
@@
 F 0 "TP28" H 6500 4200 50  0000 C BNN
 F 1 "Adc3" H 6500 4150 50  0000 C CNN
-F 2 "Measurement_Points:Measurement_Point_Round-SMD-Pad_Small" H 6500 3900 50  0001 C CNN
+F 2 "Pin_Headers:Pin_Header_Straight_1x01_Pitch2.00mm" H 6500 3900 50  0001 C CNN
 F 3 "" H 6500 3900 50  0001 C CNN
 	1    6500 3900
@@
 F 0 "TP29" H 7900 4200 50  0000 C BNN
 F 1 "Adc2" H 7900 4150 50  0000 C CNN
-F 2 "Measurement_Points:Measurement_Point_Round-SMD-Pad_Small" H 7900 3900 50  0001 C CNN
+F 2 "Pin_Headers:Pin_Header_Straight_1x01_Pitch2.00mm" H 7900 3900 50  0001 C CNN
 F 3 "" H 7900 3900 50  0001 C CNN
 	1    7900 3900
@@
 F 0 "TP30" H 9300 4200 50  0000 C BNN
 F 1 "Adc1" H 9300 4150 50  0000 C CNN
-F 2 "Measurement_Points:Measurement_Point_Round-SMD-Pad_Small" H 9300 3900 50  0001 C CNN
+F 2 "Pin_Headers:Pin_Header_Straight_1x01_Pitch2.00mm" H 9300 3900 50  0001 C CNN
 F 3 "" H 9300 3900 50  0001 C CNN
 	1    9300 3900
@@
 F 0 "TP25" H 2800 3400 50  0000 C BNN
 F 1 "AdcV" H 2800 3350 50  0000 C CNN
-F 2 "Measurement_Points:Measurement_Point_Round-SMD-Pad_Small" H 2800 3100 50  0001 C CNN
+F 2 "Pin_Headers:Pin_Header_Straight_1x01_Pitch2.00mm" H 2800 3100 50  0001 C CNN
 F 3 "" H 2800 3100 50  0001 C CNN
 	1    2800 3100
@@
 F 0 "TP26" H 2950 4100 50  0000 C BNN
 F 1 "~AdcCs" H 2950 4050 50  0000 C CNN
-F 2 "Measurement_Points:Measurement_Point_Round-SMD-Pad_Small" H 2950 3800 50  0001 C CNN
+F 2 "Pin_Headers:Pin_Header_Straight_1x01_Pitch2.00mm" H 2950 3800 50  0001 C CNN
 F 3 "" H 2950 3800 50  0001 C CNN
 	1    2950 3800
@@
 F 0 "TP24" H 2700 4100 50  0000 C BNN
 F 1 "AdcSclk" H 2700 4050 50  0000 C CNN
-F 2 "Measurement_Points:Measurement_Point_Round-SMD-Pad_Small" H 2700 3800 50  0001 C CNN
+F 2 "Pin_Headers:Pin_Header_Straight_1x01_Pitch2.00mm" H 2700 3800 50  0001 C CNN
 F 3 "" H 2700 3800 50  0001 C CNN
 	1    2700 3800
@@
 F 0 "TP23" H 2450 4100 50  0000 C BNN
 F 1 "AdcMosi" H 2450 4050 50  0000 C CNN
-F 2 "Measurement_Points:Measurement_Point_Round-SMD-Pad_Small" H 2450 3800 50  0001 C CNN
+F 2 "Pin_Headers:Pin_Header_Straight_1x01_Pitch2.00mm" H 2450 3800 50  0001 C CNN
 F 3 "" H 2450 3800 50  0001 C CNN
 	1    2450 3800
@@
 F 0 "TP22" H 2200 4100 50  0000 C BNN
 F 1 "AdcMiso" H 2200 4050 50  0000 C CNN
-F 2 "Measurement_Points:Measurement_Point_Round-SMD-Pad_Small" H 2200 3800 50  0001 C CNN
+F 2 "Pin_Headers:Pin_Header_Straight_1x01_Pitch2.00mm" H 2200 3800 50  0001 C CNN
 F 3 "" H 2200 3800 50  0001 C CNN
 	1    2200 3800

Commit message: Migrated to kicad 5
Parts:
- C27, C28, C29, C30, C31, C32: symbol C -> Device:C
- D3, D4, D5, D6: symbol D_TVS -> Device:D_TVS
- L1: symbol L -> Device:L
- R26, R27, R28, R29, R30, R31, R32, R33, R34: symbol R -> Device:R
- TP22, TP23, TP24, TP25, TP26, TP27, TP28, TP29, TP30: symbol TEST -> PrototypeBoard-rescue:TEST
- U5: symbol ADC124S021 -> PrototypeBoard-rescue:ADC124S021
Changed lines of the file:
@@
-EESchema Schematic File Version 2
-LIBS:power
-LIBS:device
-LIBS:switches
-LIBS:relays
-LIBS:motors
-LIBS:transistors
-LIBS:conn
-LIBS:linear
-LIBS:regul
-LIBS:74xx
-LIBS:cmos4000
-LIBS:adc-dac
-LIBS:memory
-LIBS:xilinx
-LIBS:microcontrollers
-LIBS:dsp
-LIBS:microchip
-LIBS:analog_switches
-LIBS:motorola
-LIBS:texas
-LIBS:intel
-LIBS:audio
-LIBS:interface
-LIBS:digital-audio
-LIBS:philips
-LIBS:display
-LIBS:cypress
-LIBS:siliconi
-LIBS:opto
-LIBS:atmel
-LIBS:contrib
-LIBS:valves
+EESchema Schematic File Version 4
 LIBS:PrototypeBoard-cache
-EELAYER 25 0
+EELAYER 26 0
 EELAYER END
 $Descr A4 11693 8268
@@
 $EndDescr
 $Comp
-L ADC124S021 U5
+L PrototypeBoard-rescue:ADC124S021 U5
 U 1 1 5AFC77A1
 P 4050 3550
@@
 ADC_IN4
 $Comp
-L L L1
+L Device:L L1
 U 1 1 5AFC781F
 P 1900 3250
@@
 $EndComp
 $Comp
-L C C28
+L Device:C C28
 U 1 1 5AFC7ED4
 P 2400 3100
@@
 $EndComp
 $Comp
-L GND #PWR047
+L power:GND #PWR047
 U 1 1 5AFC7F46
 P 2400 2950
@@
 $EndComp
 $Comp
-L C C27
+L Device:C C27
 U 1 1 5AFC7FC0
 P 2150 3100
@@
 $EndComp
 $Comp
-L GND #PWR048
+L power:GND #PWR048
 U 1 1 5AFC7FEF
 P 2150 2950
@@
 $EndComp
 $Comp
-L +3.3V #PWR049
+L power:+3.3V #PWR049
 U 1 1 5AFC801E
 P 1350 3250
@@
 Connection ~ 2400 3250
 $Comp
-L GND #PWR050
+L power:GND #PWR050
 U 1 1 5AFC8357
 P 3200 3850
@@
 	1900 3700 3200 3700
 $Comp
-L C C32
+L Device:C C32
 U 1 1 5AFD651F
 P 9900 4050
@@
 $EndComp
 $Comp
-L C C31
+L Device:C C31
 U 1 1 5AFD65A4
 P 8500 4050
@@
 $EndComp
 $Comp
-L C C30
+L Device:C C30
 U 1 1 5AFD65D2
 P 7100 4050
@@
 $EndComp
 $Comp
-L C C29
+L Device:C C29
 U 1 1 5AFD660C
 P 5700 4050
@@
 $EndComp
 $Comp
-L R R27
+L Device:R R27
 U 1 1 5AFD665A
 P 6000 3050
@@
 $EndComp
 $Comp
-L R R29
+L Device:R R29
 U 1 1 5AFD6721
 P 7400 3050
@@
 $EndComp
 $Comp
-L R R31
+L Device:R R31
 U 1 1 5AFD6757
 P 8800 3050
@@
 $EndComp
 $Comp
-L R R33
+L Device:R R33
 U 1 1 5AFD6790
 P 10200 3050
@@
 	10200 2800 10200 2900
 $Comp
-L R R34
+L Device:R R34
 U 1 1 5AFD684A
 P 10200 4050
@@
 $EndComp
 $Comp
-L R R32
+L Device:R R32
 U 1 1 5AFD68B5
 P 8800 4050
@@
 $EndComp
 $Comp
-L R R30
+L Device:R R30
 U 1 1 5AFD6903
 P 7400 4050
@@
 $EndComp
 $Comp
-L R R28
+L Device:R R28
 U 1 1 5AFD695A
 P 6000 4050
@@
 $EndComp
 $Comp
-L GND #PWR051
+L power:GND #PWR051
 U 1 1 5AFD6E2A
 P 5700 4300
@@
 $EndComp
 $Comp
-L GND #PWR052
+L power:GND #PWR052
 U 1 1 5AFD6E6C
 P 6000 4300
@@
 $EndComp
 $Comp
-L GND #PWR053
+L power:GND #PWR053
 U 1 1 5AFD6EA7
 P 7100 4300
@@
 $EndComp
 $Comp
-L GND #PWR054
+L power:GND #PWR054
 U 1 1 5AFD6EE2
 P 7400 4300
@@
 $EndComp
 $Comp
-L GND #PWR055
+L power:GND #PWR055
 U 1 1 5AFD6F1D
 P 8500 4300
@@
 $EndComp
 $Comp
-L GND #PWR056
+L power:GND #PWR056
 U 1 1 5AFD6F58
 P 8800 4300
@@
 $EndComp
 $Comp
-L GND #PWR057
+L power:GND #PWR057
 U 1 1 5AFD6F93
 P 9900 4300
@@
 $EndComp
 $Comp
-L GND #PWR058
+L power:GND #PWR058
 U 1 1 5AFD6FCE
 P 10200 4300
@@
 	10200 4200 10200 4300
 $Comp
-L TEST TP27
+L PrototypeBoard-rescue:TEST TP27
 U 1 1 5AFEFB54
 P 5100 3900
@@
 $EndComp
 $Comp
-L TEST TP28
+L PrototypeBoard-rescue:TEST TP28
 U 1 1 5AFEFBCA
 P 6500 3900
@@
 $EndComp
 $Comp
-L TEST TP29
+L PrototypeBoard-rescue:TEST TP29
 U 1 1 5AFEFC22
 P 7900 3900
@@
 $EndComp
 $Comp
-L TEST TP30
+L PrototypeBoard-rescue:TEST TP30
 U 1 1 5AFEFC7D
 P 9300 3900
@@
 $EndComp
 $Comp
-L TEST TP25
+L PrototypeBoard-rescue:TEST TP25
 U 1 1 5AFF07FE
 P 2800 3100
@@
 $EndComp
 $Comp
-L TEST TP26
+L PrototypeBoard-rescue:TEST TP26
 U 1 1 5AFF0C2E
 P 2950 3800
@@
 $EndComp
 $Comp
-L TEST TP24
+L PrototypeBoard-rescue:TEST TP24
 U 1 1 5AFF0D2B
 P 2700 3800
@@
 $EndComp
 $Comp
-L TEST TP23
+L PrototypeBoard-rescue:TEST TP23
 U 1 1 5AFF0D86
 P 2450 3800
@@
 $EndComp
 $Comp
-L TEST TP22
+L PrototypeBoard-rescue:TEST TP22
 U 1 1 5AFF0DE8
 P 2200 3800
@@
 Connection ~ 2950 3400
 $Comp
-L PWR_FLAG #FLG059
+L power:PWR_FLAG #FLG059
 U 1 1 5AFF7DCE
 P 3100 3000
@@
 	10200 3200 10200 3900
 $Comp
-L GND #PWR060
+L power:GND #PWR060
 U 1 1 5B002B6C
 P 5400 4300
@@
 $EndComp
 $Comp
-L GND #PWR061
+L power:GND #PWR061
 U 1 1 5B002BCE
 P 6800 4300
@@
 $EndComp
 $Comp
-L GND #PWR062
+L power:GND #PWR062
 U 1 1 5B002C30
 P 8200 4300
@@
 $EndComp
 $Comp
-L GND #PWR063
+L power:GND #PWR063
 U 1 1 5B002C92
 P 9600 4300
@@
 modify this part in order to use an analog hall encoder (low pass filtering, voltage divider)
 $Comp
-L D_TVS D6
+L Device:D_TVS D6
 U 1 1 5AFF1E54
 P 9600 4050
@@
 $EndComp
 $Comp
-L D_TVS D3
+L Device:D_TVS D3
 U 1 1 5AFF1F87
 P 5400 4050
@@
 $EndComp
 $Comp
-L D_TVS D4
+L Device:D_TVS D4
 U 1 1 5AFF2000
 P 6800 4050
@@
 $EndComp
 $Comp
-L D_TVS D5
+L Device:D_TVS D5
 U 1 1 5AFF208E
 P 8200 4050
@@
 $EndComp
 $Comp
-L R R26
+L Device:R R26
 U 1 1 5B210B75
 P 1550 3250
