File: Hardware/PrototypeBoard/PowerStage.sch (KiCad schematic (older format))
At the start: 20 parts, among them Q1 Q_NMOS_SGD, Q2 Q_NMOS_SGD, Q3 Q_NMOS_SGD, Q4 Q_NMOS_SGD, Q5 Q_NMOS_SGD, Q6 Q_NMOS_SGD

Commit message: Migrated to kicad 5
Parts:
- C10, C11, C12, C13, C14, C6, C7, C8, C9: symbol C -> Device:C
- C4, C5: symbol CP -> Device:CP
- Q1, Q2, Q3, Q4, Q5, Q6: symbol Q_NMOS_SGD -> Device:Q_NMOS_SGD
- TP3, TP4, TP5: symbol TEST -> PrototypeBoard-rescue:TEST
Changed lines of the file:
@@
-EESchema Schematic File Version 2
-LIBS:power
-LIBS:device
-LIBS:switches
-LIBS:relays
-LIBS:motors
-LIBS:transistors
-LIBS:conn
-LIBS:linear
-LIBS:regul
-LIBS:74xx
-LIBS:cmos4000
-LIBS:adc-dac
-LIBS:memory
-LIBS:xilinx
-LIBS:microcontrollers
-LIBS:dsp
-LIBS:microchip
-LIBS:analog_switches
-LIBS:motorola
-LIBS:texas
-LIBS:intel
-LIBS:audio
-LIBS:interface
-LIBS:digital-audio
-LIBS:philips
-LIBS:display
-LIBS:cypress
-LIBS:siliconi
-LIBS:opto
-LIBS:atmel
-LIBS:contrib
-LIBS:valves
+EESchema Schematic File Version 4
 LIBS:PrototypeBoard-cache
-EELAYER 25 0
+EELAYER 26 0
 EELAYER END
 $Descr A4 11693 8268
@@
 $EndDescr
 $Comp
-L GNDPWR #PWR012
+L PrototypeBoard-rescue:GNDPWR #PWR012
 U 1 1 56C10B12
 P 3100 4100
@@
 $EndComp
 $Comp
-L GNDPWR #PWR013
+L PrototypeBoard-rescue:GNDPWR #PWR013
 U 1 1 56C10B18
 P 5300 4100
@@
 $EndComp
 $Comp
-L GNDPWR #PWR014
+L PrototypeBoard-rescue:GNDPWR #PWR014
 U 1 1 56C10B1E
 P 7500 4100
@@
 Source_W_L
 $Comp
-L +BATT #PWR015
+L power:+BATT #PWR015
 U 1 1 56C3D45F
 P 5300 2100
@@
 $EndComp
 $Comp
-L +BATT #PWR016
+L power:+BATT #PWR016
 U 1 1 56C3D47F
 P 3100 2100
@@
 $EndComp
 $Comp
-L +BATT #PWR017
+L power:+BATT #PWR017
 U 1 1 56C3D49F
 P 7500 2100
@@
 Power_Phase_W
 $Comp
-L TEST TP3
+L PrototypeBoard-rescue:TEST TP3
 U 1 1 5B008CF2
 P 3100 2900
@@
 $EndComp
 $Comp
-L TEST TP4
+L PrototypeBoard-rescue:TEST TP4
 U 1 1 5B008D58
 P 5300 2900
@@
 $EndComp
 $Comp
-L TEST TP5
+L PrototypeBoard-rescue:TEST TP5
 U 1 1 5B008DA6
 P 7500 2900
@@
 $EndComp
 $Comp
-L C C7
+L Device:C C7
 U 1 1 5B00A350
 P 3100 4950
@@
 $EndComp
 $Comp
-L C C8
+L Device:C C8
 U 1 1 5B00A447
 P 3500 4950
@@
 $EndComp
 $Comp
-L C C6
+L Device:C C6
 U 1 1 5B00A488
 P 2700 4950
@@
 $EndComp
 $Comp
-L CP C4
+L Device:CP C4
 U 1 1 5B00A755
 P 1500 4950
@@
 $EndComp
 $Comp
-L CP C5
+L Device:CP C5
 U 1 1 5B00A808
 P 1900 4950
@@
 $EndComp
 $Comp
-L GNDPWR #PWR018
+L PrototypeBoard-rescue:GNDPWR #PWR018
 U 1 1 5B00BA7D
 P 3100 5300
@@
 $EndComp
 $Comp
-L GNDPWR #PWR019
+L PrototypeBoard-rescue:GNDPWR #PWR019
 U 1 1 5B00BB28
 P 5300 5300
@@
 $EndComp
 $Comp
-L GNDPWR #PWR020
+L PrototypeBoard-rescue:GNDPWR #PWR020
 U 1 1 5B00BB6F
 P 7500 5300
@@
 $EndComp
 $Comp
-L GNDPWR #PWR021
+L PrototypeBoard-rescue:GNDPWR #PWR021
 U 1 1 5B00BBB6
 P 1700 5300
@@
 Connection ~ 1700 5200
 $Comp
-L +BATT #PWR022
+L power:+BATT #PWR022
 U 1 1 5B00C18C
 P 3100 4600
@@
 $EndComp
 $Comp
-L +BATT #PWR023
+L power:+BATT #PWR023
 U 1 1 5B00C1D3
 P 5300 4600
@@
 $EndComp
 $Comp
-L +BATT #PWR024
+L power:+BATT #PWR024
 U 1 1 5B00C21A
 P 7500 4600
@@
 $EndComp
 $Comp
-L C C9
+L Device:C C9
 U 1 1 5B00C673
 P 4900 4950
@@
 $EndComp
 $Comp
-L C C11
+L Device:C C11
 U 1 1 5B00C6D6
 P 5700 4950
@@
 $EndComp
 $Comp
-L C C12
+L Device:C C12
 U 1 1 5B00C72E
 P 7100 4950
@@
 $EndComp
 $Comp
-L C C14
+L Device:C C14
 U 1 1 5B00C79B
 P 7900 4950
@@
 $EndComp
 $Comp
-L C C10
+L Device:C C10
 U 1 1 5B00C7FB
 P 5300 4950
@@
 $EndComp
 $Comp
-L C C13
+L Device:C C13
 U 1 1 5B00C86E
 P 7500 4950
@@
 $EndComp
 $Comp
-L +BATT #PWR025
+L power:+BATT #PWR025
 U 1 1 5B00C9A4
 P 1700 4600
@@
 Connection ~ 1700 4700
 $Comp
-L Q_NMOS_SGD Q1
+L Device:Q_NMOS_SGD Q1
 U 1 1 5B00718F
 P 3000 2400
@@
 $EndComp
 $Comp
-L Q_NMOS_SGD Q2
+L Device:Q_NMOS_SGD Q2
 U 1 1 5B00724E
 P 3000 3600
@@
 $EndComp
 $Comp
-L Q_NMOS_SGD Q4
+L Device:Q_NMOS_SGD Q4
 U 1 1 5B0072F2
 P 5200 3600
@@
 $EndComp
 $Comp
-L Q_NMOS_SGD Q3
+L Device:Q_NMOS_SGD Q3
 U 1 1 5B007385
 P 5200 2400
@@
 $EndComp
 $Comp
-L Q_NMOS_SGD Q5
+L Device:Q_NMOS_SGD Q5
 U 1 1 5B0073FB
 P 7400 2400
@@
 $EndComp
 $Comp
-L Q_NMOS_SGD Q6
+L Device:Q_NMOS_SGD Q6
 U 1 1 5B00749A
 P 7400 3600

Commit message: New, much bigger pcb layout, changes to connection PGND <-> GND
Parts:
- added NT1, NT2, NT3: Net-Tie_2, symbol Device:Net-Tie_2
Connections:
- net labels added: GND
- wire segments 56 -> 88
Changed lines of the file:
@@
 $EndDescr
 $Comp
-L PrototypeBoard-rescue:GNDPWR #PWR012
+L PrototypeBoard-rescue:GNDPWR #PWR019
 U 1 1 56C10B12
 P 3100 4100
-F 0 "#PWR012" H 3100 3900 50  0001 C CNN
+F 0 "#PWR019" H 3100 3900 50  0001 C CNN
 F 1 "GNDPWR" H 3100 3970 50  0000 C CNN
 F 2 "" H 3100 4050 50  0000 C CNN
@@
 $EndComp
 $Comp
-L PrototypeBoard-rescue:GNDPWR #PWR013
+L PrototypeBoard-rescue:GNDPWR #PWR023
 U 1 1 56C10B18
 P 5300 4100
-F 0 "#PWR013" H 5300 3900 50  0001 C CNN
+F 0 "#PWR023" H 5300 3900 50  0001 C CNN
 F 1 "GNDPWR" H 5300 3970 50  0000 C CNN
 F 2 "" H 5300 4050 50  0000 C CNN
@@
 $EndComp
 $Comp
-L PrototypeBoard-rescue:GNDPWR #PWR014
+L PrototypeBoard-rescue:GNDPWR #PWR027
 U 1 1 56C10B1E
 P 7500 4100
-F 0 "#PWR014" H 7500 3900 50  0001 C CNN
+F 0 "#PWR027" H 7500 3900 50  0001 C CNN
 F 1 "GNDPWR" H 7500 3970 50  0000 C CNN
 F 2 "" H 7500 4050 50  0000 C CNN
@@
 Source_W_L
 $Comp
-L power:+BATT #PWR015
+L power:+BATT #PWR022
 U 1 1 56C3D45F
 P 5300 2100
-F 0 "#PWR015" H 5300 1950 50  0001 C CNN
+F 0 "#PWR022" H 5300 1950 50  0001 C CNN
 F 1 "+BATT" H 5300 2240 50  0000 C CNN
 F 2 "" H 5300 2100 50  0000 C CNN
@@
 $EndComp
 $Comp
-L power:+BATT #PWR016
+L power:+BATT #PWR018
 U 1 1 56C3D47F
 P 3100 2100
-F 0 "#PWR016" H 3100 1950 50  0001 C CNN
+F 0 "#PWR018" H 3100 1950 50  0001 C CNN
 F 1 "+BATT" H 3100 2240 50  0000 C CNN
 F 2 "" H 3100 2100 50  0000 C CNN
@@
 $EndComp
 $Comp
-L power:+BATT #PWR017
+L power:+BATT #PWR026
 U 1 1 56C3D49F
 P 7500 2100
-F 0 "#PWR017" H 7500 1950 50  0001 C CNN
+F 0 "#PWR026" H 7500 1950 50  0001 C CNN
 F 1 "+BATT" H 7500 2240 50  0000 C CNN
 F 2 "" H 7500 2100 50  0000 C CNN
@@
 $EndComp
 $Comp
-L PrototypeBoard-rescue:GNDPWR #PWR018
+L PrototypeBoard-rescue:GNDPWR #PWR021
 U 1 1 5B00BA7D
 P 3100 5300
-F 0 "#PWR018" H 3100 5100 50  0001 C CNN
+F 0 "#PWR021" H 3100 5100 50  0001 C CNN
 F 1 "GNDPWR" H 3100 5170 50  0000 C CNN
 F 2 "" H 3100 5250 50  0000 C CNN
@@
 $EndComp
 $Comp
-L PrototypeBoard-rescue:GNDPWR #PWR019
+L PrototypeBoard-rescue:GNDPWR #PWR025
 U 1 1 5B00BB28
 P 5300 5300
-F 0 "#PWR019" H 5300 5100 50  0001 C CNN
+F 0 "#PWR025" H 5300 5100 50  0001 C CNN
 F 1 "GNDPWR" H 5300 5170 50  0000 C CNN
 F 2 "" H 5300 5250 50  0000 C CNN
@@
 $EndComp
 $Comp
-L PrototypeBoard-rescue:GNDPWR #PWR020
+L PrototypeBoard-rescue:GNDPWR #PWR029
 U 1 1 5B00BB6F
 P 7500 5300
-F 0 "#PWR020" H 7500 5100 50  0001 C CNN
+F 0 "#PWR029" H 7500 5100 50  0001 C CNN
 F 1 "GNDPWR" H 7500 5170 50  0000 C CNN
 F 2 "" H 7500 5250 50  0000 C CNN
@@
 $EndComp
 $Comp
-L PrototypeBoard-rescue:GNDPWR #PWR021
+L PrototypeBoard-rescue:GNDPWR #PWR017
 U 1 1 5B00BBB6
 P 1700 5300
-F 0 "#PWR021" H 1700 5100 50  0001 C CNN
+F 0 "#PWR017" H 1700 5100 50  0001 C CNN
 F 1 "GNDPWR" H 1700 5170 50  0000 C CNN
 F 2 "" H 1700 5250 50  0000 C CNN
@@
 $EndComp
 Wire Wire Line
-	3100 2600 3100 3400
-Wire Wire Line
-	5300 2600 5300 3400
-Wire Wire Line
-	7500 2600 7500 3400
+	3100 2600 3100 2700
+Wire Wire Line
+	5300 2600 5300 2700
+Wire Wire Line
+	7500 2600 7500 2700
 Wire Wire Line
 	3100 2900 3200 2900
@@
 	7500 2100 7500 2200
 Wire Wire Line
-	3100 4100 3100 3800
-Wire Wire Line
-	5300 4100 5300 3800
-Wire Wire Line
-	7500 4100 7500 3800
-Wire Wire Line
-	7100 5200 7900 5200
-Wire Wire Line
-	4900 5200 5700 5200
-Wire Wire Line
-	2700 5200 3500 5200
-Wire Wire Line
-	2700 4700 3500 4700
-Wire Wire Line
-	4900 4700 5700 4700
-Wire Wire Line
-	7100 4700 7900 4700
-Wire Wire Line
-	1500 4700 1900 4700
-Wire Wire Line
-	1500 5200 1900 5200
+	7100 5200 7500 5200
+Wire Wire Line
+	4900 5200 5300 5200
+Wire Wire Line
+	2700 5200 3100 5200
+Wire Wire Line
+	2700 4700 3100 4700
+Wire Wire Line
+	4900 4700 5300 4700
+Wire Wire Line
+	7100 4700 7500 4700
+Wire Wire Line
+	1500 4700 1700 4700
+Wire Wire Line
+	1500 5200 1700 5200
 Wire Wire Line
 	2700 4800 2700 4700
@@
 	2700 5200 2700 5100
 Wire Wire Line
-	3100 5100 3100 5300
+	3100 5100 3100 5200
 Connection ~ 3100 5200
 Wire Wire Line
-	3100 4600 3100 4800
+	3100 4600 3100 4700
 Connection ~ 3100 4700
 Wire Wire Line
@@
 	4900 5100 4900 5200
 Wire Wire Line
-	5300 5100 5300 5300
+	5300 5100 5300 5200
 Connection ~ 5300 5200
 Wire Wire Line
-	5300 4600 5300 4800
+	5300 4600 5300 4700
 Connection ~ 5300 4700
 Wire Wire Line
@@
 	7100 5100 7100 5200
 Wire Wire Line
-	7500 5100 7500 5300
+	7500 5100 7500 5200
 Connection ~ 7500 5200
 Wire Wire Line
-	7500 4600 7500 4800
+	7500 4600 7500 4700
 Connection ~ 7500 4700
 Wire Wire Line
@@
 Connection ~ 1700 5200
 $Comp
-L power:+BATT #PWR022
+L power:+BATT #PWR020
 U 1 1 5B00C18C
 P 3100 4600
-F 0 "#PWR022" H 3100 4450 50  0001 C CNN
+F 0 "#PWR020" H 3100 4450 50  0001 C CNN
 F 1 "+BATT" H 3100 4740 50  0000 C CNN
 F 2 "" H 3100 4600 50  0000 C CNN
@@
 $EndComp
 $Comp
-L power:+BATT #PWR023
+L power:+BATT #PWR024
 U 1 1 5B00C1D3
 P 5300 4600
-F 0 "#PWR023" H 5300 4450 50  0001 C CNN
+F 0 "#PWR024" H 5300 4450 50  0001 C CNN
 F 1 "+BATT" H 5300 4740 50  0000 C CNN
 F 2 "" H 5300 4600 50  0000 C CNN
@@
 $EndComp
 $Comp
-L power:+BATT #PWR024
+L power:+BATT #PWR028
 U 1 1 5B00C21A
 P 7500 4600
-F 0 "#PWR024" H 7500 4450 50  0001 C CNN
+F 0 "#PWR028" H 7500 4450 50  0001 C CNN
 F 1 "+BATT" H 7500 4740 50  0000 C CNN
 F 2 "" H 7500 4600 50  0000 C CNN
@@
 $EndComp
 $Comp
-L power:+BATT #PWR025
+L power:+BATT #PWR016
 U 1 1 5B00C9A4
 P 1700 4600
-F 0 "#PWR025" H 1700 4450 50  0001 C CNN
+F 0 "#PWR016" H 1700 4450 50  0001 C CNN
 F 1 "+BATT" H 1700 4740 50  0000 C CNN
 F 2 "" H 1700 4600 50  0000 C CNN
@@
 	2700 3600 2800 3600
 Wire Wire Line
-	2700 3900 3100 3900
-Connection ~ 3100 3900
-Wire Wire Line
 	4900 2400 5000 2400
 Wire Wire Line
@@
 	4900 3600 5000 3600
 Wire Wire Line
-	4900 3900 5300 3900
-Connection ~ 5300 3900
-Wire Wire Line
 	7100 2400 7200 2400
 Wire Wire Line
@@
 	7100 3600 7200 3600
 Wire Wire Line
-	7100 3900 7500 3900
+	3100 2900 3100 3400
+Wire Wire Line
+	5300 2900 5300 3400
+Wire Wire Line
+	7500 2900 7500 3400
+Wire Wire Line
+	3100 5200 3500 5200
+Wire Wire Line
+	3100 5200 3100 5300
+Wire Wire Line
+	3100 4700 3500 4700
+Wire Wire Line
+	3100 4700 3100 4800
+Wire Wire Line
+	5300 5200 5700 5200
+Wire Wire Line
+	5300 5200 5300 5300
+Wire Wire Line
+	5300 4700 5700 4700
+Wire Wire Line
+	5300 4700 5300 4800
+Wire Wire Line
+	7500 5200 7900 5200
+Wire Wire Line
+	7500 5200 7500 5300
+Wire Wire Line
+	7500 4700 7900 4700
+Wire Wire Line
+	7500 4700 7500 4800
+Wire Wire Line
+	1700 5200 1900 5200
+Wire Wire Line
+	1700 4700 1900 4700
+Wire Wire Line
+	3100 2700 3100 2900
+Wire Wire Line
+	5300 2700 5300 2900
+Wire Wire Line
+	7500 2700 7500 2900
+$Comp
+L Device:Net-Tie_2 NT3
+U 1 1 5B89D5DC
+P 7300 3900
+F 0 "NT3" H 7300 4078 50  0000 C CNN
+F 1 "Net-Tie_2" H 7300 3987 50  0000 C CNN
+F 2 "" H 7300 3900 50  0001 C CNN
+F 3 "~" H 7300 3900 50  0001 C CNN
+	1    7300 3900
+	1    0    0    -1
+$EndComp
+Wire Wire Line
+	7500 3800 7500 3900
+$Comp
+L Device:Net-Tie_2 NT2
+U 1 1 5B89D8FA
+P 5100 3900
+F 0 "NT2" H 5100 4078 50  0000 C CNN
+F 1 "Net-Tie_2" H 5100 3987 50  0000 C CNN
+F 2 "" H 5100 3900 50  0001 C CNN
+F 3 "~" H 5100 3900 50  0001 C CNN
+	1    5100 3900
+	1    0    0    -1
+$EndComp
+$Comp
+L Device:Net-Tie_2 NT1
+U 1 1 5B89D9AA
+P 2900 3900
+F 0 "NT1" H 2900 4078 50  0000 C CNN
+F 1 "Net-Tie_2" H 2900 3987 50  0000 C CNN
+F 2 "" H 2900 3900 50  0001 C CNN
+F 3 "~" H 2900 3900 50  0001 C CNN
+	1    2900 3900
+	1    0    0    -1
+$EndComp
+Wire Wire Line
+	5300 3800 5300 3900
+Wire Wire Line
+	3100 3800 3100 3900
+Wire Wire Line
+	5200 3900 5300 3900
+Connection ~ 5300 3900
+Wire Wire Line
+	5300 3900 5300 4100
+Wire Wire Line
+	4900 3900 4950 3900
+Wire Wire Line
+	3000 3900 3100 3900
+Connection ~ 3100 3900
+Wire Wire Line
+	3100 3900 3100 4100
+Wire Wire Line
+	2700 3900 2750 3900
+Wire Wire Line
+	7400 3900 7500 3900
 Connection ~ 7500 3900
+Wire Wire Line
+	7500 3900 7500 4100
+Wire Wire Line
+	7100 3900 7150 3900
+$Comp
+L power:GND #PWR?
+U 1 1 5B8A7A9D
+P 4950 4100
+AR Path="/56D57CF9/5B8A7A9D" Ref="#PWR?"  Part="1"
+AR Path="/56D57CF9/56D58A10/5B8A7A9D" Ref="#PWR0101"  Part="1"
+F 0 "#PWR0101" H 4950 3850 50  0001 C CNN
+F 1 "GND" H 4950 3950 50  0000 C CNN
+F 2 "" H 4950 4100 50  0001 C CNN
+F 3 "" H 4950 4100 50  0001 C CNN
+	1    4950 4100
+	1    0    0    -1
+$EndComp
+$Comp
+L power:GND #PWR?
+U 1 1 5B8A9701
+P 2750 4100
+AR Path="/56D57CF9/5B8A9701" Ref="#PWR?"  Part="1"
+AR Path="/56D57CF9/56D58A10/5B8A9701" Ref="#PWR0102"  Part="1"
+F 0 "#PWR0102" H 2750 3850 50  0001 C CNN
+F 1 "GND" H 2750 3950 50  0000 C CNN
+F 2 "" H 2750 4100 50  0001 C CNN
+F 3 "" H 2750 4100 50  0001 C CNN
+	1    2750 4100
+	1    0    0    -1
+$EndComp
+$Comp
+L power:GND #PWR?
+U 1 1 5B8AB37D
+P 7150 4100
+AR Path="/56D57CF9/5B8AB37D" Ref="#PWR?"  Part="1"
+AR Path="/56D57CF9/56D58A10/5B8AB37D" Ref="#PWR0103"  Part="1"
+F 0 "#PWR0103" H 7150 3850 50  0001 C CNN
+F 1 "GND" H 7150 3950 50  0000 C CNN
+F 2 "" H 7150 4100 50  0001 C CNN
+F 3 "" H 7150 4100 50  0001 C CNN
+	1    7150 4100
+	1    0    0    -1
+$EndComp
+Wire Wire Line
+	7150 3900 7150 4100
+Connection ~ 7150 3900
+Wire Wire Line
+	7150 3900 7200 3900
+Wire Wire Line
+	4950 3900 4950 4100
+Connection ~ 4950 3900
+Wire Wire Line
+	4950 3900 5000 3900
+Wire Wire Line
+	2750 3900 2750 4100
+Connection ~ 2750 3900
+Wire Wire Line
+	2750 3900 2800 3900
 $EndSCHEMATC

Commit message: continued to work on new layout
Parts:
- NT1, NT2, NT3: footprint (none) -> NetTie:NetTie-2_SMD_Pad0.5mm
Changed lines of the file:
@@
 F 0 "NT3" H 7300 4078 50  0000 C CNN
 F 1 "Net-Tie_2" H 7300 3987 50  0000 C CNN
-F 2 "" H 7300 3900 50  0001 C CNN
+F 2 "NetTie:NetTie-2_SMD_Pad0.5mm" H 7300 3900 50  0001 C CNN
 F 3 "~" H 7300 3900 50  0001 C CNN
 	1    7300 3900
@@
 F 0 "NT2" H 5100 4078 50  0000 C CNN
 F 1 "Net-Tie_2" H 5100 3987 50  0000 C CNN
-F 2 "" H 5100 3900 50  0001 C CNN
+F 2 "NetTie:NetTie-2_SMD_Pad0.5mm" H 5100 3900 50  0001 C CNN
 F 3 "~" H 5100 3900 50  0001 C CNN
 	1    5100 3900
@@
 F 0 "NT1" H 2900 4078 50  0000 C CNN
 F 1 "Net-Tie_2" H 2900 3987 50  0000 C CNN
-F 2 "" H 2900 3900 50  0001 C CNN
+F 2 "NetTie:NetTie-2_SMD_Pad0.5mm" H 2900 3900 50  0001 C CNN
 F 3 "~" H 2900 3900 50  0001 C CNN
 	1    2900 3900

Commit message: Gate driver closer to power stage, ground and power ground seperated completely, power ground traces to gate driver replaced by power planes, phase outputs now span across all layers (vias not places yet)
Parts:
- removed NT1, NT2, NT3: Net-Tie_2, NetTie:NetTie-2_SMD_Pad0.5mm, symbol Device:Net-Tie_2
Connections:
- net labels removed: GND
- wire segments 88 -> 79
Changed lines of the file:
@@
 Wire Wire Line
 	7500 2700 7500 2900
-$Comp
-L Device:Net-Tie_2 NT3
-U 1 1 5B89D5DC
-P 7300 3900
-F 0 "NT3" H 7300 4078 50  0000 C CNN
-F 1 "Net-Tie_2" H 7300 3987 50  0000 C CNN
-F 2 "NetTie:NetTie-2_SMD_Pad0.5mm" H 7300 3900 50  0001 C CNN
-F 3 "~" H 7300 3900 50  0001 C CNN
-	1    7300 3900
-	1    0    0    -1
-$EndComp
 Wire Wire Line
 	7500 3800 7500 3900
-$Comp
-L Device:Net-Tie_2 NT2
-U 1 1 5B89D8FA
-P 5100 3900
-F 0 "NT2" H 5100 4078 50  0000 C CNN
-F 1 "Net-Tie_2" H 5100 3987 50  0000 C CNN
-F 2 "NetTie:NetTie-2_SMD_Pad0.5mm" H 5100 3900 50  0001 C CNN
-F 3 "~" H 5100 3900 50  0001 C CNN
-	1    5100 3900
-	1    0    0    -1
-$EndComp
-$Comp
-L Device:Net-Tie_2 NT1
-U 1 1 5B89D9AA
-P 2900 3900
-F 0 "NT1" H 2900 4078 50  0000 C CNN
-F 1 "Net-Tie_2" H 2900 3987 50  0000 C CNN
-F 2 "NetTie:NetTie-2_SMD_Pad0.5mm" H 2900 3900 50  0001 C CNN
-F 3 "~" H 2900 3900 50  0001 C CNN
-	1    2900 3900
-	1    0    0    -1
-$EndComp
 Wire Wire Line
 	5300 3800 5300 3900
 Wire Wire Line
 	3100 3800 3100 3900
-Wire Wire Line
-	5200 3900 5300 3900
 Connection ~ 5300 3900
 Wire Wire Line
 	5300 3900 5300 4100
-Wire Wire Line
-	4900 3900 4950 3900
-Wire Wire Line
-	3000 3900 3100 3900
 Connection ~ 3100 3900
 Wire Wire Line
 	3100 3900 3100 4100
-Wire Wire Line
-	2700 3900 2750 3900
-Wire Wire Line
-	7400 3900 7500 3900
 Connection ~ 7500 3900
 Wire Wire Line
 	7500 3900 7500 4100
 Wire Wire Line
-	7100 3900 7150 3900
-$Comp
-L power:GND #PWR?
-U 1 1 5B8A7A9D
-P 4950 4100
-AR Path="/56D57CF9/5B8A7A9D" Ref="#PWR?"  Part="1"
-AR Path="/56D57CF9/56D58A10/5B8A7A9D" Ref="#PWR0101"  Part="1"
-F 0 "#PWR0101" H 4950 3850 50  0001 C CNN
-F 1 "GND" H 4950 3950 50  0000 C CNN
-F 2 "" H 4950 4100 50  0001 C CNN
-F 3 "" H 4950 4100 50  0001 C CNN
-	1    4950 4100
-	1    0    0    -1
-$EndComp
-$Comp
-L power:GND #PWR?
-U 1 1 5B8A9701
-P 2750 4100
-AR Path="/56D57CF9/5B8A9701" Ref="#PWR?"  Part="1"
-AR Path="/56D57CF9/56D58A10/5B8A9701" Ref="#PWR0102"  Part="1"
-F 0 "#PWR0102" H 2750 3850 50  0001 C CNN
-F 1 "GND" H 2750 3950 50  0000 C CNN
-F 2 "" H 2750 4100 50  0001 C CNN
-F 3 "" H 2750 4100 50  0001 C CNN
-	1    2750 4100
-	1    0    0    -1
-$EndComp
-$Comp
-L power:GND #PWR?
-U 1 1 5B8AB37D
-P 7150 4100
-AR Path="/56D57CF9/5B8AB37D" Ref="#PWR?"  Part="1"
-AR Path="/56D57CF9/56D58A10/5B8AB37D" Ref="#PWR0103"  Part="1"
-F 0 "#PWR0103" H 7150 3850 50  0001 C CNN
-F 1 "GND" H 7150 3950 50  0000 C CNN
-F 2 "" H 7150 4100 50  0001 C CNN
-F 3 "" H 7150 4100 50  0001 C CNN
-	1    7150 4100
-	1    0    0    -1
-$EndComp
+	4900 3900 5300 3900
 Wire Wire Line
-	7150 3900 7150 4100
-Connection ~ 7150 3900
+	2700 3900 3100 3900
 Wire Wire Line
-	7150 3900 7200 3900
-Wire Wire Line
-	4950 3900 4950 4100
-Connection ~ 4950 3900
-Wire Wire Line
-	4950 3900 5000 3900
-Wire Wire Line
-	2750 3900 2750 4100
-Connection ~ 2750 3900
-Wire Wire Line
-	2750 3900 2800 3900
+	7100 3900 7500 3900
 $EndSCHEMATC

Commit message: All tracks routed, fixed bug in schematic, smaller test points
Parts:
- TP3, TP4, TP5: footprint Pin_Headers:Pin_Header_Straight_1x01_Pitch2.00mm -> Pin_Headers:Pin_Header_Straight_1x01_Pitch1.00mm
Changed lines of the file:
@@
 F 0 "TP3" H 3100 3200 50  0000 C BNN
 F 1 "PhaseU" H 3100 3150 50  0000 C CNN
-F 2 "Pin_Headers:Pin_Header_Straight_1x01_Pitch2.00mm" H 3100 2900 50  0001 C CNN
+F 2 "Pin_Headers:Pin_Header_Straight_1x01_Pitch1.00mm" H 3100 2900 50  0001 C CNN
 F 3 "" H 3100 2900 50  0001 C CNN
 	1    3100 2900
@@
 F 0 "TP4" H 5300 3200 50  0000 C BNN
 F 1 "PhaseV" H 5300 3150 50  0000 C CNN
-F 2 "Pin_Headers:Pin_Header_Straight_1x01_Pitch2.00mm" H 5300 2900 50  0001 C CNN
+F 2 "Pin_Headers:Pin_Header_Straight_1x01_Pitch1.00mm" H 5300 2900 50  0001 C CNN
 F 3 "" H 5300 2900 50  0001 C CNN
 	1    5300 2900
@@
 F 0 "TP5" H 7500 3200 50  0000 C BNN
 F 1 "PhaseW" H 7500 3150 50  0000 C CNN
-F 2 "Pin_Headers:Pin_Header_Straight_1x01_Pitch2.00mm" H 7500 2900 50  0001 C CNN
+F 2 "Pin_Headers:Pin_Header_Straight_1x01_Pitch1.00mm" H 7500 2900 50  0001 C CNN
 F 3 "" H 7500 2900 50  0001 C CNN
 	1    7500 2900
