File: Hardware/PrototypeBoard/EncoderConnector.sch (KiCad schematic (older format))
At the start: 9 parts, among them J2 Encoder

Commit message: assigned net classes and a few net names
Parts:
- JP4, JP5, JP6, JP7: footprint Connectors:PINHEAD1-3 -> Connectors:GS3
Changed lines of the file:
@@
 F 0 "JP4" H 4400 2150 50  0000 L CNN
 F 1 "SPI/Hall" H 4350 2350 50  0000 C BNN
-F 2 "Connectors:PINHEAD1-3" H 4350 2250 50  0001 C CNN
+F 2 "Connectors:GS3" H 4350 2250 50  0001 C CNN
 F 3 "" H 4350 2250 50  0001 C CNN
 	1    4350 2250
@@
 F 0 "JP5" H 4400 2450 50  0000 L CNN
 F 1 "SPI/Hall" H 4350 2650 50  0000 C BNN
-F 2 "Connectors:PINHEAD1-3" H 4350 2550 50  0001 C CNN
+F 2 "Connectors:GS3" H 4350 2550 50  0001 C CNN
 F 3 "" H 4350 2550 50  0001 C CNN
 	1    4350 2550
@@
 F 0 "JP6" H 7750 2050 50  0000 L CNN
 F 1 "SPI/Hall" H 7700 2250 50  0000 C BNN
-F 2 "Connectors:PINHEAD1-3" H 7700 2150 50  0001 C CNN
+F 2 "Connectors:GS3" H 7700 2150 50  0001 C CNN
 F 3 "" H 7700 2150 50  0001 C CNN
 	1    7700 2150
@@
 F 0 "JP7" H 7750 2350 50  0000 L CNN
 F 1 "SPI/Hall" H 7700 2550 50  0000 C BNN
-F 2 "Connectors:PINHEAD1-3" H 7700 2450 50  0001 C CNN
+F 2 "Connectors:GS3" H 7700 2450 50  0001 C CNN
 F 3 "" H 7700 2450 50  0001 C CNN
 	1    7700 2450

Commit message: minor progress in layout
Parts:
- TP31, TP32, TP33, TP34: footprint Measurement_Points:Measurement_Point_Round-TH_Big -> Measurement_Points:Measurement_Point_Round-SMD-Pad_Small
Changed lines of the file:
@@
 F 0 "TP31" H 5300 2600 50  0000 C BNN
 F 1 "EncSclk/HallA" H 5300 2550 50  0000 C CNN
-F 2 "Measurement_Points:Measurement_Point_Round-TH_Big" H 5300 2300 50  0001 C CNN
+F 2 "Measurement_Points:Measurement_Point_Round-SMD-Pad_Small" H 5300 2300 50  0001 C CNN
 F 3 "" H 5300 2300 50  0001 C CNN
 	1    5300 2300
@@
 F 0 "TP32" H 5300 2800 50  0000 C BNN
 F 1 "!EncCs/HallB" H 5300 2750 50  0000 C CNN
-F 2 "Measurement_Points:Measurement_Point_Round-TH_Big" H 5300 2500 50  0001 C CNN
+F 2 "Measurement_Points:Measurement_Point_Round-SMD-Pad_Small" H 5300 2500 50  0001 C CNN
 F 3 "" H 5300 2500 50  0001 C CNN
 	1    5300 2500
@@
 F 0 "TP34" H 6900 2700 50  0000 C BNN
 F 1 "EncMiso/HallC" H 6900 2650 50  0000 C CNN
-F 2 "Measurement_Points:Measurement_Point_Round-TH_Big" H 6900 2400 50  0001 C CNN
+F 2 "Measurement_Points:Measurement_Point_Round-SMD-Pad_Small" H 6900 2400 50  0001 C CNN
 F 3 "" H 6900 2400 50  0001 C CNN
 	1    6900 2400
@@
 F 0 "TP33" H 6900 2500 50  0000 C BNN
 F 1 "EncMosi/NC" H 6900 2450 50  0000 C CNN
-F 2 "Measurement_Points:Measurement_Point_Round-TH_Big" H 6900 2200 50  0001 C CNN
+F 2 "Measurement_Points:Measurement_Point_Round-SMD-Pad_Small" H 6900 2200 50  0001 C CNN
 F 3 "" H 6900 2200 50  0001 C CNN
 	1    6900 2200

Commit message: more layout and some changes to schematic
Parts:
- removed J2: Encoder, Pin_Headers:Pin_Header_Straight_1x06_Pitch2.54mm, symbol Conn_02x03_Odd_Even
- added C33: 100n, Capacitors_SMD:C_0805_HandSoldering, symbol C
- added J2: Conn_01x06, Pin_Headers:Pin_Header_Straight_1x06_Pitch2.00mm, symbol Conn_01x06
- TP31: renamed from TP32; footprint Measurement_Points:Measurement_Point_Round-SMD-Pad_Small -> Pin_Headers:Pin_Header_Straight_1x01_Pitch2.00mm
- TP32: renamed from TP34; footprint Measurement_Points:Measurement_Point_Round-SMD-Pad_Small -> Pin_Headers:Pin_Header_Straight_1x01_Pitch2.00mm
- TP33: renamed from TP31; footprint Measurement_Points:Measurement_Point_Round-SMD-Pad_Small -> Pin_Headers:Pin_Header_Straight_1x01_Pitch2.00mm
- TP34: renamed from TP33; footprint Measurement_Points:Measurement_Point_Round-SMD-Pad_Small -> Pin_Headers:Pin_Header_Straight_1x01_Pitch2.00mm
- renumbered JP5 to JP4, JP7 to JP5, JP4 to JP6, JP6 to JP7
Connections:
- wire segments 8 -> 6
Changed lines of the file:
@@
 $EndDescr
-$Comp
-L Conn_02x03_Odd_Even J2
-U 1 1 5AFC940D
-P 6000 2350
-F 0 "J2" H 6050 2550 50  0000 C CNN
-F 1 "Encoder" H 6050 2150 50  0000 C CNN
-F 2 "Pin_Headers:Pin_Header_Straight_1x06_Pitch2.54mm" H 6000 2350 50  0001 C CNN
-F 3 "" H 6000 2350 50  0001 C CNN
-	1    6000 2350
-	1    0    0    -1
-$EndComp
 $Comp
 L GND #PWR064
 U 1 1 5AFC9462
-P 5800 2250
-F 0 "#PWR064" H 5800 2000 50  0001 C CNN
-F 1 "GND" H 5800 2100 50  0000 C CNN
-F 2 "" H 5800 2250 50  0001 C CNN
-F 3 "" H 5800 2250 50  0001 C CNN
-	1    5800 2250
+P 9750 2900
+F 0 "#PWR064" H 9750 2650 50  0001 C CNN
+F 1 "GND" H 9750 2750 50  0000 C CNN
+F 2 "" H 9750 2900 50  0001 C CNN
+F 3 "" H 9750 2900 50  0001 C CNN
+	1    9750 2900
 	0    1    1    0
 $EndComp
@@
 L +3.3V #PWR065
 U 1 1 5AFC948F
-P 6300 2450
-F 0 "#PWR065" H 6300 2300 50  0001 C CNN
-F 1 "+3.3V" H 6300 2590 50  0000 C CNN
-F 2 "" H 6300 2450 50  0001 C CNN
-F 3 "" H 6300 2450 50  0001 C CNN
-	1    6300 2450
-	0    1    1    0
+P 9800 3400
+F 0 "#PWR065" H 9800 3250 50  0001 C CNN
+F 1 "+3.3V" H 9800 3540 50  0000 C CNN
+F 2 "" H 9800 3400 50  0001 C CNN
+F 3 "" H 9800 3400 50  0001 C CNN
+	1    9800 3400
+	0    -1   -1   0
 $EndComp
-Text HLabel 4600 2250 2    60   Input ~ 0
+Text HLabel 9150 2900 2    60   Input ~ 0
 SCLK
-Text HLabel 4100 2550 0    60   Input ~ 0
+Text HLabel 7550 3000 2    60   Input ~ 0
 ~CS
-Text HLabel 7450 2450 0    60   Output ~ 0
+Text HLabel 4350 3200 2    60   Output ~ 0
 MISO
-Text HLabel 7450 2150 0    60   Input ~ 0
+Text HLabel 5950 3100 2    60   Input ~ 0
 MOSI
-Text HLabel 4100 2250 0    60   Output ~ 0
+Text HLabel 8650 2900 0    60   Output ~ 0
 HALL_A
-Text HLabel 4600 2550 2    60   Output ~ 0
+Text HLabel 7050 3000 0    60   Output ~ 0
 HALL_B
 $Comp
+L Jumper_NC_Dual JP6
+U 1 1 5AFC952B
+P 7300 3000
+F 0 "JP6" H 7350 2900 50  0000 L CNN
+F 1 "SPI/Hall" H 7300 3100 50  0000 C BNN
+F 2 "Connectors:GS3" H 7300 3000 50  0001 C CNN
+F 3 "" H 7300 3000 50  0001 C CNN
+	1    7300 3000
+	1    0    0    -1
+$EndComp
+$Comp
 L Jumper_NC_Dual JP4
-U 1 1 5AFC952B
-P 4350 2250
-F 0 "JP4" H 4400 2150 50  0000 L CNN
-F 1 "SPI/Hall" H 4350 2350 50  0000 C BNN
-F 2 "Connectors:GS3" H 4350 2250 50  0001 C CNN
-F 3 "" H 4350 2250 50  0001 C CNN
-	1    4350 2250
+U 1 1 5AFC9571
+P 4100 3200
+F 0 "JP4" H 4150 3100 50  0000 L CNN
+F 1 "SPI/Hall" H 4100 3300 50  0000 C BNN
+F 2 "Connectors:GS3" H 4100 3200 50  0001 C CNN
+F 3 "" H 4100 3200 50  0001 C CNN
+	1    4100 3200
+	1    0    0    -1
+$EndComp
+$Comp
+L Jumper_NC_Dual JP7
+U 1 1 5AFC95E5
+P 8900 2900
+F 0 "JP7" H 8950 2800 50  0000 L CNN
+F 1 "SPI/Hall" H 8900 3000 50  0000 C BNN
+F 2 "Connectors:GS3" H 8900 2900 50  0001 C CNN
+F 3 "" H 8900 2900 50  0001 C CNN
+	1    8900 2900
 	1    0    0    -1
 $EndComp
 $Comp
 L Jumper_NC_Dual JP5
-U 1 1 5AFC9571
-P 4350 2550
-F 0 "JP5" H 4400 2450 50  0000 L CNN
-F 1 "SPI/Hall" H 4350 2650 50  0000 C BNN
-F 2 "Connectors:GS3" H 4350 2550 50  0001 C CNN
-F 3 "" H 4350 2550 50  0001 C CNN
-	1    4350 2550
-	-1   0    0    1
-$EndComp
-$Comp
-L Jumper_NC_Dual JP6
-U 1 1 5AFC95E5
-P 7700 2150
-F 0 "JP6" H 7750 2050 50  0000 L CNN
-F 1 "SPI/Hall" H 7700 2250 50  0000 C BNN
-F 2 "Connectors:GS3" H 7700 2150 50  0001 C CNN
-F 3 "" H 7700 2150 50  0001 C CNN
-	1    7700 2150
+U 1 1 5AFC9628
+P 5700 3100
+F 0 "JP5" H 5750 3000 50  0000 L CNN
+F 1 "SPI/Hall" H 5700 3200 50  0000 C BNN
+F 2 "Connectors:GS3" H 5700 3100 50  0001 C CNN
+F 3 "" H 5700 3100 50  0001 C CNN
+	1    5700 3100
 	1    0    0    -1
 $EndComp
 $Comp
-L Jumper_NC_Dual JP7
-U 1 1 5AFC9628
-P 7700 2450
-F 0 "JP7" H 7750 2350 50  0000 L CNN
-F 1 "SPI/Hall" H 7700 2550 50  0000 C BNN
-F 2 "Connectors:GS3" H 7700 2450 50  0001 C CNN
-F 3 "" H 7700 2450 50  0001 C CNN
-	1    7700 2450
-	-1   0    0    1
+L GND #PWR066
+U 1 1 5AFC9686
+P 3850 3200
+F 0 "#PWR066" H 3850 2950 50  0001 C CNN
+F 1 "GND" H 3850 3050 50  0000 C CNN
+F 2 "" H 3850 3200 50  0001 C CNN
+F 3 "" H 3850 3200 50  0001 C CNN
+	1    3850 3200
+	0    1    1    0
+$EndComp
+Text HLabel 5450 3100 0    60   Output ~ 0
+HALL_C
+$Comp
+L TEST TP33
+U 1 1 5AFF16A3
+P 6700 3100
+F 0 "TP33" H 6700 3400 50  0000 C BNN
+F 1 "EncSclk/HallA" H 6700 3350 50  0000 C CNN
+F 2 "Pin_Headers:Pin_Header_Straight_1x01_Pitch2.00mm" H 6700 3100 50  0001 C CNN
+F 3 "" H 6700 3100 50  0001 C CNN
+	1    6700 3100
+	0    -1   -1   0
+$EndComp
+$Comp
+L TEST TP31
+U 1 1 5AFF1700
+P 3450 3300
+F 0 "TP31" H 3450 3600 50  0000 C BNN
+F 1 "!EncCs/HallB" H 3450 3550 50  0000 C CNN
+F 2 "Pin_Headers:Pin_Header_Straight_1x01_Pitch2.00mm" H 3450 3300 50  0001 C CNN
+F 3 "" H 3450 3300 50  0001 C CNN
+	1    3450 3300
+	0    -1   -1   0
+$EndComp
+$Comp
+L TEST TP32
+U 1 1 5AFF1757
+P 5100 3200
+F 0 "TP32" H 5100 3500 50  0000 C BNN
+F 1 "EncMiso/HallC" H 5100 3450 50  0000 C CNN
+F 2 "Pin_Headers:Pin_Header_Straight_1x01_Pitch2.00mm" H 5100 3200 50  0001 C CNN
+F 3 "" H 5100 3200 50  0001 C CNN
+	1    5100 3200
+	0    -1   -1   0
+$EndComp
+$Comp
+L TEST TP34
+U 1 1 5AFF17C5
+P 8300 3000
+F 0 "TP34" H 8300 3300 50  0000 C BNN
+F 1 "EncMosi/NC" H 8300 3250 50  0000 C CNN
+F 2 "Pin_Headers:Pin_Header_Straight_1x01_Pitch2.00mm" H 8300 3000 50  0001 C CNN
+F 3 "" H 8300 3000 50  0001 C CNN
+	1    8300 3000
+	0    -1   -1   0
+$EndComp
+$Comp
+L Conn_01x06 J2
+U 1 1 5B245F83
+P 10100 3100
+F 0 "J2" H 10100 3400 50  0000 C CNN
+F 1 "Conn_01x06" H 10100 2700 50  0000 C CNN
+F 2 "Pin_Headers:Pin_Header_Straight_1x06_Pitch2.00mm" H 10100 3100 50  0001 C CNN
+F 3 "" H 10100 3100 50  0001 C CNN
+	1    10100 3100
+	1    0    0    -1
 $EndComp
 Wire Wire Line
-	4350 2350 5800 2350
+	9750 2900 9900 2900
 Wire Wire Line
-	4350 2450 5800 2450
+	8300 3000 9900 3000
+Connection ~ 8900 3000
 Wire Wire Line
-	6300 2350 7700 2350
+	6700 3100 9900 3100
+Connection ~ 7300 3100
 Wire Wire Line
-	6300 2250 7700 2250
+	5100 3200 9900 3200
+Connection ~ 5700 3200
+Wire Wire Line
+	3450 3300 9900 3300
+Connection ~ 4100 3300
+Wire Wire Line
+	9900 3400 9800 3400
 $Comp
-L GND #PWR066
-U 1 1 5AFC9686
-P 7950 2150
-F 0 "#PWR066" H 7950 1900 50  0001 C CNN
-F 1 "GND" H 7950 2000 50  0000 C CNN
-F 2 "" H 7950 2150 50  0001 C CNN
-F 3 "" H 7950 2150 50  0001 C CNN
-	1    7950 2150
-	0    -1   -1   0
-$EndComp
-Text HLabel 7950 2450 2    60   Output ~ 0
-HALL_C
-$Comp
-L TEST TP31
-U 1 1 5AFF16A3
-P 5300 2300
-F 0 "TP31" H 5300 2600 50  0000 C BNN
-F 1 "EncSclk/HallA" H 5300 2550 50  0000 C CNN
-F 2 "Measurement_Points:Measurement_Point_Round-SMD-Pad_Small" H 5300 2300 50  0001 C CNN
-F 3 "" H 5300 2300 50  0001 C CNN
-	1    5300 2300
+L +3.3V #PWR067
+U 1 1 5B247C3F
+P 10400 3000
+F 0 "#PWR067" H 10400 2850 50  0001 C CNN
+F 1 "+3.3V" H 10400 3140 50  0000 C CNN
+F 2 "" H 10400 3000 50  0001 C CNN
+F 3 "" H 10400 3000 50  0001 C CNN
+	1    10400 3000
 	1    0    0    -1
 $EndComp
 $Comp
-L TEST TP32
-U 1 1 5AFF1700
-P 5300 2500
-F 0 "TP32" H 5300 2800 50  0000 C BNN
-F 1 "!EncCs/HallB" H 5300 2750 50  0000 C CNN
-F 2 "Measurement_Points:Measurement_Point_Round-SMD-Pad_Small" H 5300 2500 50  0001 C CNN
-F 3 "" H 5300 2500 50  0001 C CNN
-	1    5300 2500
-	-1   0    0    1
+L GND #PWR068
+U 1 1 5B247C68
+P 10400 3300
+F 0 "#PWR068" H 10400 3050 50  0001 C CNN
+F 1 "GND" H 10400 3150 50  0000 C CNN
+F 2 "" H 10400 3300 50  0001 C CNN
+F 3 "" H 10400 3300 50  0001 C CNN
+	1    10400 3300
+	1    0    0    -1
 $EndComp
 $Comp
-L TEST TP34
-U 1 1 5AFF1757
-P 6900 2400
-F 0 "TP34" H 6900 2700 50  0000 C BNN
-F 1 "EncMiso/HallC" H 6900 2650 50  0000 C CNN
-F 2 "Measurement_Points:Measurement_Point_Round-SMD-Pad_Small" H 6900 2400 50  0001 C CNN
-F 3 "" H 6900 2400 50  0001 C CNN
-	1    6900 2400
-	-1   0    0    1
-$EndComp
-$Comp
-L TEST TP33
-U 1 1 5AFF17C5
-P 6900 2200
-F 0 "TP33" H 6900 2500 50  0000 C BNN
-F 1 "EncMosi/NC" H 6900 2450 50  0000 C CNN
-F 2 "Measurement_Points:Measurement_Point_Round-SMD-Pad_Small" H 6900 2200 50  0001 C CNN
-F 3 "" H 6900 2200 50  0001 C CNN
-	1    6900 2200
+L C C33
+U 1 1 5B247DBB
+P 10400 3150
+F 0 "C33" H 10425 3250 50  0000 L CNN
+F 1 "100n" H 10425 3050 50  0000 L CNN
+F 2 "Capacitors_SMD:C_0805_HandSoldering" H 10438 3000 50  0001 C CNN
+F 3 "" H 10400 3150 50  0001 C CNN
+	1    10400 3150
 	1    0    0    -1
 $EndComp
-Wire Wire Line
-	5300 2300 5300 2350
-Connection ~ 5300 2350
-Wire Wire Line
-	5300 2500 5300 2450
-Connection ~ 5300 2450
-Wire Wire Line
-	6900 2400 6900 2350
-Connection ~ 6900 2350
-Wire Wire Line
-	6900 2200 6900 2250
-Connection ~ 6900 2250
 $EndSCHEMATC

Commit message: Migrated to kicad 5
Parts:
- C33: symbol C -> Device:C
- J2: symbol Conn_01x06 -> conn:Conn_01x06
- JP4, JP5, JP6, JP7: symbol Jumper_NC_Dual -> Device:Jumper_NC_Dual
- TP31, TP32, TP33, TP34: symbol TEST -> PrototypeBoard-rescue:TEST
Changed lines of the file:
@@
-EESchema Schematic File Version 2
-LIBS:power
-LIBS:device
-LIBS:switches
-LIBS:relays
-LIBS:motors
-LIBS:transistors
-LIBS:conn
-LIBS:linear
-LIBS:regul
-LIBS:74xx
-LIBS:cmos4000
-LIBS:adc-dac
-LIBS:memory
-LIBS:xilinx
-LIBS:microcontrollers
-LIBS:dsp
-LIBS:microchip
-LIBS:analog_switches
-LIBS:motorola
-LIBS:texas
-LIBS:intel
-LIBS:audio
-LIBS:interface
-LIBS:digital-audio
-LIBS:philips
-LIBS:display
-LIBS:cypress
-LIBS:siliconi
-LIBS:opto
-LIBS:atmel
-LIBS:contrib
-LIBS:valves
+EESchema Schematic File Version 4
 LIBS:PrototypeBoard-cache
-EELAYER 25 0
+EELAYER 26 0
 EELAYER END
 $Descr A4 11693 8268
@@
 $EndDescr
 $Comp
-L GND #PWR064
+L power:GND #PWR064
 U 1 1 5AFC9462
 P 9750 2900
@@
 $EndComp
 $Comp
-L +3.3V #PWR065
+L power:+3.3V #PWR065
 U 1 1 5AFC948F
 P 9800 3400
@@
 HALL_B
 $Comp
-L Jumper_NC_Dual JP6
+L Device:Jumper_NC_Dual JP6
 U 1 1 5AFC952B
 P 7300 3000
@@
 $EndComp
 $Comp
-L Jumper_NC_Dual JP4
+L Device:Jumper_NC_Dual JP4
 U 1 1 5AFC9571
 P 4100 3200
@@
 $EndComp
 $Comp
-L Jumper_NC_Dual JP7
+L Device:Jumper_NC_Dual JP7
 U 1 1 5AFC95E5
 P 8900 2900
@@
 $EndComp
 $Comp
-L Jumper_NC_Dual JP5
+L Device:Jumper_NC_Dual JP5
 U 1 1 5AFC9628
 P 5700 3100
@@
 $EndComp
 $Comp
-L GND #PWR066
+L power:GND #PWR066
 U 1 1 5AFC9686
 P 3850 3200
@@
 HALL_C
 $Comp
-L TEST TP33
+L PrototypeBoard-rescue:TEST TP33
 U 1 1 5AFF16A3
 P 6700 3100
@@
 $EndComp
 $Comp
-L TEST TP31
+L PrototypeBoard-rescue:TEST TP31
 U 1 1 5AFF1700
 P 3450 3300
@@
 $EndComp
 $Comp
-L TEST TP32
+L PrototypeBoard-rescue:TEST TP32
 U 1 1 5AFF1757
 P 5100 3200
@@
 $EndComp
 $Comp
-L TEST TP34
+L PrototypeBoard-rescue:TEST TP34
 U 1 1 5AFF17C5
 P 8300 3000
@@
 $EndComp
 $Comp
-L Conn_01x06 J2
+L conn:Conn_01x06 J2
 U 1 1 5B245F83
 P 10100 3100
@@
 	9900 3400 9800 3400
 $Comp
-L +3.3V #PWR067
+L power:+3.3V #PWR067
 U 1 1 5B247C3F
 P 10400 3000
@@
 $EndComp
 $Comp
-L GND #PWR068
+L power:GND #PWR068
 U 1 1 5B247C68
 P 10400 3300
@@
 $EndComp
 $Comp
-L C C33
+L Device:C C33
 U 1 1 5B247DBB
 P 10400 3150

Commit message: Added LEDs for PWM, SPI communication, Gate Driver Errors and Gate Driver disabled
Connections:
- wire segments 6 -> 10
Changed lines of the file:
@@
 $EndDescr
 $Comp
-L power:GND #PWR067
+L power:GND #PWR073
 U 1 1 5AFC9462
 P 9750 2900
-F 0 "#PWR067" H 9750 2650 50  0001 C CNN
+F 0 "#PWR073" H 9750 2650 50  0001 C CNN
 F 1 "GND" H 9750 2750 50  0000 C CNN
 F 2 "" H 9750 2900 50  0001 C CNN
@@
 $EndComp
 $Comp
-L power:+3.3V #PWR068
+L power:+3.3V #PWR074
 U 1 1 5AFC948F
 P 9800 3400
-F 0 "#PWR068" H 9800 3250 50  0001 C CNN
+F 0 "#PWR074" H 9800 3250 50  0001 C CNN
 F 1 "+3.3V" H 9800 3540 50  0000 C CNN
 F 2 "" H 9800 3400 50  0001 C CNN
@@
 $EndComp
 $Comp
-L power:GND #PWR066
+L power:GND #PWR072
 U 1 1 5AFC9686
 P 3850 3200
-F 0 "#PWR066" H 3850 2950 50  0001 C CNN
+F 0 "#PWR072" H 3850 2950 50  0001 C CNN
 F 1 "GND" H 3850 3050 50  0000 C CNN
 F 2 "" H 3850 3200 50  0001 C CNN
@@
 	9750 2900 9900 2900
 Wire Wire Line
-	8300 3000 9900 3000
+	8300 3000 8900 3000
 Connection ~ 8900 3000
 Wire Wire Line
-	6700 3100 9900 3100
+	6700 3100 7300 3100
 Connection ~ 7300 3100
 Wire Wire Line
-	5100 3200 9900 3200
+	5100 3200 5700 3200
 Connection ~ 5700 3200
 Wire Wire Line
-	3450 3300 9900 3300
+	3450 3300 4100 3300
 Connection ~ 4100 3300
 Wire Wire Line
 	9900 3400 9800 3400
 $Comp
-L power:+3.3V #PWR069
+L power:+3.3V #PWR075
 U 1 1 5B247C3F
 P 10400 3000
-F 0 "#PWR069" H 10400 2850 50  0001 C CNN
+F 0 "#PWR075" H 10400 2850 50  0001 C CNN
 F 1 "+3.3V" H 10400 3140 50  0000 C CNN
 F 2 "" H 10400 3000 50  0001 C CNN
@@
 $EndComp
 $Comp
-L power:GND #PWR070
+L power:GND #PWR076
 U 1 1 5B247C68
 P 10400 3300
-F 0 "#PWR070" H 10400 3050 50  0001 C CNN
+F 0 "#PWR076" H 10400 3050 50  0001 C CNN
 F 1 "GND" H 10400 3150 50  0000 C CNN
 F 2 "" H 10400 3300 50  0001 C CNN
@@
 	1    0    0    -1
 $EndComp
+Wire Wire Line
+	8900 3000 9900 3000
+Wire Wire Line
+	7300 3100 9900 3100
+Wire Wire Line
+	5700 3200 9900 3200
+Wire Wire Line
+	4100 3300 9900 3300
 $EndSCHEMATC

Commit message: All tracks routed, fixed bug in schematic, smaller test points
Parts:
- TP31, TP32: footprint Pin_Headers:Pin_Header_Straight_1x01_Pitch2.00mm -> Pin_Headers:Pin_Header_Straight_1x01_Pitch1.00mm
Changed lines of the file:
@@
 F 0 "TP31" H 3450 3600 50  0000 C BNN
 F 1 "!EncCs/HallB" H 3450 3550 50  0000 C CNN
-F 2 "Pin_Headers:Pin_Header_Straight_1x01_Pitch2.00mm" H 3450 3300 50  0001 C CNN
+F 2 "Pin_Headers:Pin_Header_Straight_1x01_Pitch1.00mm" H 3450 3300 50  0001 C CNN
 F 3 "" H 3450 3300 50  0001 C CNN
 	1    3450 3300
@@
 F 0 "TP32" H 5100 3500 50  0000 C BNN
 F 1 "EncMiso/HallC" H 5100 3450 50  0000 C CNN
-F 2 "Pin_Headers:Pin_Header_Straight_1x01_Pitch2.00mm" H 5100 3200 50  0001 C CNN
+F 2 "Pin_Headers:Pin_Header_Straight_1x01_Pitch1.00mm" H 5100 3200 50  0001 C CNN
 F 3 "" H 5100 3200 50  0001 C CNN
 	1    5100 3200

Commit message: Some deduplication, renaming and cleanups in the schematic
Connections:
- net labels added: HallA, HallB, HallC, Miso, Mosi, Sclk, ~Cs
- net labels removed: HALL_A, HALL_B, HALL_C, MISO, MOSI, SCLK, ~CS
Changed lines of the file:
@@
 $Descr A4 11693 8268
 encoding utf-8
-Sheet 7 8
+Sheet 7 13
 Title ""
 Date ""
@@
 $EndComp
 Text HLabel 9150 2900 2    60   Input ~ 0
-SCLK
+Sclk
 Text HLabel 7550 3000 2    60   Input ~ 0
-~CS
+~Cs
 Text HLabel 4350 3200 2    60   Output ~ 0
-MISO
+Miso
 Text HLabel 5950 3100 2    60   Input ~ 0
-MOSI
+Mosi
 Text HLabel 8650 2900 0    60   Output ~ 0
-HALL_A
+HallA
 Text HLabel 7050 3000 0    60   Output ~ 0
-HALL_B
+HallB
 $Comp
 L Device:Jumper_NC_Dual JP6
@@
 $EndComp
 Text HLabel 5450 3100 0    60   Output ~ 0
-HALL_C
+HallC
 $Comp
 L PrototypeBoard-rescue:TEST TP33
