File: Hardware/PrototypeBoard/PrototypeBoard.sch (KiCad schematic (older format))
At the start: 10 parts

Commit message: All tracks routed, fixed bug in schematic, smaller test points
Parts:
- TP1, TP2: footprint Pin_Headers:Pin_Header_Straight_1x01_Pitch2.00mm -> Pin_Headers:Pin_Header_Straight_1x01_Pitch1.00mm
Changed lines of the file:
@@
 F 0 "TP2" H 10400 2000 50  0000 C BNN
 F 1 "5.5-28V" H 10400 1950 50  0000 C CNN
-F 2 "Pin_Headers:Pin_Header_Straight_1x01_Pitch2.00mm" H 10400 1700 50  0001 C CNN
+F 2 "Pin_Headers:Pin_Header_Straight_1x01_Pitch1.00mm" H 10400 1700 50  0001 C CNN
 F 3 "" H 10400 1700 50  0001 C CNN
 	1    10400 1700
@@
 F 0 "TP1" H 9800 2000 50  0000 C BNN
 F 1 "3.3V" H 9800 1950 50  0000 C CNN
-F 2 "Pin_Headers:Pin_Header_Straight_1x01_Pitch2.00mm" H 9800 1700 50  0001 C CNN
+F 2 "Pin_Headers:Pin_Header_Straight_1x01_Pitch1.00mm" H 9800 1700 50  0001 C CNN
 F 3 "" H 9800 1700 50  0001 C CNN
 	1    9800 1700
